Commit message: Harmonic
Signed-off-by: Juancams <jc.manzanares.serrano@gmail.com>

File: pal_robotiq_description/urdf/robotiq_140_gripper.urdf.xacro (robot description, xacro)
@@ -32,5 +32,5 @@
         <origin xyz="0 0 0" rpy="0 0 0" />
         <geometry>
-          <mesh filename="package://pal_robotiq_description/meshes/visual/robotiq_${stroke}_outer_knuckle.stl" />
+          <mesh filename="file://$(find pal_robotiq_description)/meshes/visual/robotiq_${stroke}_outer_knuckle.stl" />
         </geometry>
         <material name="">
@@ -41,5 +41,5 @@
         <origin xyz="0 0 0" rpy="0 0 0" />
         <geometry>
-          <mesh filename="package://pal_robotiq_description/meshes/collision/robotiq_${stroke}_outer_knuckle.stl" />
+          <mesh filename="file://$(find pal_robotiq_description)/meshes/collision/robotiq_${stroke}_outer_knuckle.stl" />
         </geometry>
       </collision>
@@ -58,5 +58,5 @@
         <origin xyz="0 0 0" rpy="0 0 0" />
         <geometry>
-          <mesh filename="package://pal_robotiq_description/meshes/visual/robotiq_${stroke}_outer_finger.stl" />
+          <mesh filename="file://$(find pal_robotiq_description)/meshes/visual/robotiq_${stroke}_outer_finger.stl" />
         </geometry>
         <material name="">
@@ -67,5 +67,5 @@
         <origin xyz="0 0 0" rpy="0 0 0" />
         <geometry>
-          <mesh filename="package://pal_robotiq_description/meshes/collision/robotiq_${stroke}_outer_finger.stl" />
+          <mesh filename="file://$(find pal_robotiq_description)/meshes/collision/robotiq_${stroke}_outer_finger.stl" />
         </geometry>
       </collision>
@@ -87,5 +87,5 @@
         <origin xyz="0 0 0" rpy="0 0 0" />
         <geometry>
-          <mesh filename="package://pal_robotiq_description/meshes/visual/robotiq_${stroke}_inner_knuckle.stl" />
+          <mesh filename="file://$(find pal_robotiq_description)/meshes/visual/robotiq_${stroke}_inner_knuckle.stl" />
         </geometry>
         <material name="">
@@ -96,5 +96,5 @@
         <origin xyz="0 0 0" rpy="0 0 0" />
         <geometry>
-          <mesh filename="package://pal_robotiq_description/meshes/collision/robotiq_${stroke}_inner_knuckle.stl" />
+          <mesh filename="file://$(find pal_robotiq_description)/meshes/collision/robotiq_${stroke}_inner_knuckle.stl" />
         </geometry>
       </collision>
@@ -123,5 +123,5 @@
         <origin xyz="0 0 0" rpy="0 0 0" />
         <geometry>
-          <mesh filename="package://pal_robotiq_description/meshes/visual/robotiq_${stroke}_inner_finger.stl" />
+          <mesh filename="file://$(find pal_robotiq_description)/meshes/visual/robotiq_${stroke}_inner_finger.stl" />
         </geometry>
         <material name="">
@@ -132,5 +132,5 @@
         <origin xyz="0 0 0" rpy="0 0 0" />
         <geometry>
-          <mesh filename="package://pal_robotiq_description/meshes/collision/robotiq_${stroke}_inner_finger.stl" />
+          <mesh filename="file://$(find pal_robotiq_description)/meshes/collision/robotiq_${stroke}_inner_finger.stl" />
         </geometry>
       </collision>
@@ -233,5 +233,5 @@
         <origin xyz="0 0 0" rpy="0 0 0" />
         <geometry>
-          <mesh filename="package://pal_robotiq_description/meshes/visual/robotiq_base_link.stl" />
+          <mesh filename="file://$(find pal_robotiq_description)/meshes/visual/robotiq_base_link.stl" />
         </geometry>
         <material name="">
@@ -242,5 +242,5 @@
         <origin xyz="0 0 0" rpy="0 0 0" />
         <geometry>
-          <mesh filename="package://pal_robotiq_description/meshes/collision/robotiq_base_link.stl" />
+          <mesh filename="file://$(find pal_robotiq_description)/meshes/collision/robotiq_base_link.stl" />
         </geometry>
       </collision>
@@ -255,5 +255,5 @@
           <origin xyz="0 0 0.0" rpy="3.1416 0 0" />
           <geometry>
-              <mesh filename="package://pal_robotiq_description/meshes/visual/pal_robotiq_coupling.stl"/>
+              <mesh filename="file://$(find pal_robotiq_description)/meshes/visual/pal_robotiq_coupling.stl"/>
           </geometry>
           <material name="">
@@ -264,5 +264,5 @@
           <origin xyz="0 0 0.0" rpy="3.1416 0 0" />
           <geometry>
-              <mesh filename="package://pal_robotiq_description/meshes/visual/pal_robotiq_coupling.stl"/>
+              <mesh filename="file://$(find pal_robotiq_description)/meshes/visual/pal_robotiq_coupling.stl"/>
           </geometry>
       </collision>

File: pal_robotiq_description/urdf/robotiq_85_gripper.urdf.xacro (robot description, xacro)
@@ -31,5 +31,5 @@
         <origin xyz="0 0 0" rpy="0 0 0" />
         <geometry>
-          <mesh filename="package://pal_robotiq_description/meshes/visual/robotiq_85_outer_knuckle.dae" scale="0.001 0.001 0.001"/>
+          <mesh filename="file://$(find pal_robotiq_description)/meshes/visual/robotiq_85_outer_knuckle.dae" scale="0.001 0.001 0.001"/>
         </geometry>
         <material name="">
@@ -40,5 +40,5 @@
         <origin xyz="0 0 0" rpy="0 0 0" />
         <geometry>
-          <mesh filename="package://pal_robotiq_description/meshes/collision/robotiq_85_outer_knuckle.dae" scale="0.001 0.001 0.001"/>
+          <mesh filename="file://$(find pal_robotiq_description)/meshes/collision/robotiq_85_outer_knuckle.dae" scale="0.001 0.001 0.001"/>
         </geometry>
       </collision>
@@ -57,5 +57,5 @@
         <origin xyz="0 0 0" rpy="0 0 0" />
         <geometry>
-          <mesh filename="package://pal_robotiq_description/meshes/visual/robotiq_85_outer_finger.dae" scale="0.001 0.001 0.001"/>
+          <mesh filename="file://$(find pal_robotiq_description)/meshes/visual/robotiq_85_outer_finger.dae" scale="0.001 0.001 0.001"/>
         </geometry>
         <material name="">
@@ -66,5 +66,5 @@
         <origin xyz="0 0 0" rpy="0 0 0" />
         <geometry>
-          <mesh filename="package://pal_robotiq_description/meshes/collision/robotiq_85_outer_finger.dae" scale="0.001 0.001 0.001"/>
+          <mesh filename="file://$(find pal_robotiq_description)/meshes/collision/robotiq_85_outer_finger.dae" scale="0.001 0.001 0.001"/>
         </geometry>
       </collision>
@@ -86,5 +86,5 @@
         <origin xyz="0 0 0" rpy="0 0 0" />
         <geometry>
-          <mesh filename="package://pal_robotiq_description/meshes/visual/robotiq_85_inner_knuckle.dae" scale="0.001 0.001 0.001"/>
+          <mesh filename="file://$(find pal_robotiq_description)/meshes/visual/robotiq_85_inner_knuckle.dae" scale="0.001 0.001 0.001"/>
         </geometry>
         <material name="">
@@ -95,5 +95,5 @@
         <origin xyz="0 0 0" rpy="0 0 0" />
         <geometry>
-          <mesh filename="package://pal_robotiq_description/meshes/collision/robotiq_85_inner_knuckle.dae" scale="0.001 0.001 0.001"/>
+          <mesh filename="file://$(find pal_robotiq_description)/meshes/collision/robotiq_85_inner_knuckle.dae" scale="0.001 0.001 0.001"/>
         </geometry>
       </collision>
@@ -122,5 +122,5 @@
         <origin xyz="0 0 0" rpy="0 0 0" />
         <geometry>
-          <mesh filename="package://pal_robotiq_description/meshes/visual/robotiq_85_inner_finger.dae" scale="0.001 0.001 0.001"/>
+          <mesh filename="file://$(find pal_robotiq_description)/meshes/visual/robotiq_85_inner_finger.dae" scale="0.001 0.001 0.001"/>
         </geometry>
         <material name="">
@@ -131,5 +131,5 @@
         <origin xyz="0 0 0" rpy="0 0 0" />
         <geometry>
-          <mesh filename="package://pal_robotiq_description/meshes/collision/robotiq_85_inner_finger.dae" scale="0.001 0.001 0.001" />
+          <mesh filename="file://$(find pal_robotiq_description)/meshes/collision/robotiq_85_inner_finger.dae" scale="0.001 0.001 0.001" />
         </geometry>
       </collision>
@@ -244,5 +244,5 @@
         <origin xyz="0 0 0" rpy="0 0 0" />
         <geometry>
-          <mesh filename="package://pal_robotiq_description/meshes/visual/robotiq_base_link.stl"/>
+          <mesh filename="file://$(find pal_robotiq_description)/meshes/visual/robotiq_base_link.stl"/>
         </geometry>
         <material name="">
@@ -253,5 +253,5 @@
         <origin xyz="0 0 0" rpy="0 0 0" />
         <geometry>
-          <mesh filename="package://pal_robotiq_description/meshes/collision/robotiq_base_link.stl" />
+          <mesh filename="file://$(find pal_robotiq_description)/meshes/collision/robotiq_base_link.stl" />
         </geometry>
       </collision>
@@ -266,5 +266,5 @@
           <origin xyz="0 0 0.0" rpy="3.1416 0 0" />
           <geometry>
-              <mesh filename="package://pal_robotiq_description/meshes/visual/pal_robotiq_coupling.stl"/>
+              <mesh filename="file://$(find pal_robotiq_description)/meshes/visual/pal_robotiq_coupling.stl"/>
           </geometry>
           <material name="">
@@ -275,5 +275,5 @@
           <origin xyz="0 0 0.0" rpy="3.1416 0 0" />
           <geometry>
-              <mesh filename="package://pal_robotiq_description/meshes/visual/pal_robotiq_coupling.stl"/>
+              <mesh filename="file://$(find pal_robotiq_description)/meshes/visual/pal_robotiq_coupling.stl"/>
           </geometry>
       </collision>
